File: TMC2130/TMC2130.kicad_sch (KiCad schematic)
At the start: 23 parts, among them J1 DIAG, Q1 BCX56, U1 TMC2130-TA

Commit message: changed to 6L
deleted 2 ground pours to allow for 8L assembly on JLCPCB
Parts:
- C1: LCSC (none) -> C23733
- C2: LCSC (none) -> C47339
- C3: value 470nF/16V -> 220nF/16V; LCSC (none) -> C16772
- C4: value 22nF/63V -> 22nF/50V; LCSC (none) -> C1532
- C5, C6, C7: LCSC (none) -> C307331
- D1: LCSC (none) -> C8062
- Q1: LCSC (none) -> C100026
- R1, R2: LCSC (none) -> C17168
- R3: LCSC (none) -> C25765
- R4: LCSC (none) -> C25768
- R5: value 2.2R -> 1R; LCSC (none) -> C25086
- R6: LCSC (none) -> C25076
- R7, R8: LCSC (none) -> C53899
Changed lines of the file:
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@@
+      (effects (font (size 1.27 1.27)) hide)
+    )
+    (property "LCSC" "C17168" (id 4) (at 24.765 95.885 0)
       (effects (font (size 1.27 1.27)) hide)
     )
@@
       (effects (font (size 1.27 1.27)) hide)
     )
+    (property "LCSC" "C53899" (id 4) (at 159.385 109.22 0)
+      (effects (font (size 1.27 1.27)) hide)
+    )
     (pin "1")
     (pin "2")
@@
       (effects (font (size 1.27 1.27)) hide)
     )
+    (property "LCSC" "C25076" (id 4) (at 74.295 64.77 0)
+      (effects (font (size 1.27 1.27)) hide)
+    )
     (pin "1")
     (pin "2")
@@
     )
     (property "Datasheet" "~" (id 3) (at 39.37 96.52 0)
+      (effects (font (size 1.27 1.27)) hide)
+    )
+    (property "LCSC" "C17168" (id 4) (at 39.37 96.52 0)
       (effects (font (size 1.27 1.27)) hide)
     )
@@
       (effects (font (size 1.27 1.27)) hide)
     )
+    (property "LCSC" "C25768" (id 4) (at 62.23 52.07 0)
+      (effects (font (size 1.27 1.27)) hide)
+    )
     (pin "1")
     (pin "2")
@@
       (effects (font (size 1.27 1.27)) hide)
     )
+    (property "LCSC" "C25765" (id 4) (at 52.705 93.345 0)
+      (effects (font (size 1.27 1.27)) hide)
+    )
     (pin "1")
     (pin "2")
@@
       (effects (font (size 1.27 1.27)) hide)
     )
+    (property "LCSC" "C307331" (id 4) (at 156.845 52.07 0)
+      (effects (font (size 1.27 1.27)) hide)
+    )
     (pin "1")
     (pin "2")
@@
       (effects (font (size 1.27 1.27)) (justify left))
     )
-    (property "Value" "2.2R" (id 1) (at 73.66 24.7649 0)
+    (property "Value" "1R" (id 1) (at 73.66 24.7649 0)
       (effects (font (size 1.27 1.27)) (justify left))
     )
@@
     )
     (property "Datasheet" "~" (id 3) (at 71.12 23.495 0)
+      (effects (font (size 1.27 1.27)) hide)
+    )
+    (property "LCSC" "C25086" (id 4) (at 71.12 23.495 0)
       (effects (font (size 1.27 1.27)) hide)
     )
@@
       (effects (font (size 1.27 1.27)) (justify left))
     )
-    (property "Value" "470nF/16V" (id 1) (at 77.47 73.0312 0)
+    (property "Value" "220nF/16V" (id 1) (at 77.47 73.0312 0)
       (effects (font (size 1.27 1.27)) (justify left))
     )
@@
     )
     (property "Datasheet" "~" (id 3) (at 74.295 71.755 0)
+      (effects (font (size 1.27 1.27)) hide)
+    )
+    (property "LCSC" "C16772" (id 4) (at 74.295 71.755 0)
       (effects (font (size 1.27 1.27)) hide)
     )
@@
       (effects (font (size 1.27 1.27)) (justify right))
     )
-    (property "Value" "22nF/63V" (id 1) (at 95.885 69.215 0)
+    (property "Value" "22nF/50V" (id 1) (at 95.885 69.215 0)
       (effects (font (size 1.27 1.27)) (justify right))
     )
@@
     )
     (property "Datasheet" "~" (id 3) (at 106.68 67.31 0)
+      (effects (font (size 1.27 1.27)) hide)
+    )
+    (property "LCSC" "C1532" (id 4) (at 106.68 67.31 0)
       (effects (font (size 1.27 1.27)) hide)
     )
@@
       (effects (font (size 1.27 1.27)) (justify left) hide)
     )
+    (property "LCSC" "C100026" (id 4) (at 71.755 55.88 0)
+      (effects (font (size 1.27 1.27)) hide)
+    )
     (pin "1")
     (pin "2")
@@
       (effects (font (size 1.27 1.27)) hide)
     )
+    (property "LCSC" "C8062" (id 4) (at 62.23 60.96 0)
+      (effects (font (size 1.27 1.27)) hide)
+    )
     (pin "1")
     (pin "2")
@@
     )
     (property "Datasheet" "~" (id 3) (at 71.12 29.845 0)
+      (effects (font (size 1.27 1.27)) hide)
+    )
+    (property "LCSC" "C47339" (id 4) (at 71.12 29.845 0)
       (effects (font (size 1.27 1.27)) hide)
     )
@@
       (effects (font (size 1.27 1.27)) hide)
     )
+    (property "LCSC" "C307331" (id 4) (at 146.05 52.07 0)
+      (effects (font (size 1.27 1.27)) hide)
+    )
     (pin "1")
     (pin "2")
@@
       (effects (font (size 1.27 1.27)) hide)
     )
+    (property "LCSC" "C53899" (id 4) (at 159.385 111.76 0)
+      (effects (font (size 1.27 1.27)) hide)
+    )
     (pin "1")
     (pin "2")
@@
       (effects (font (size 1.27 1.27)) hide)
     )
+    (property "LCSC" "C23733" (id 4) (at 60.96 26.67 0)
+      (effects (font (size 1.27 1.27)) hide)
+    )
     (pin "1")
     (pin "2")
@@
     )
     (property "Datasheet" "~" (id 3) (at 114.935 59.69 0)
+      (effects (font (size 1.27 1.27)) hide)
+    )
+    (property "LCSC" "C307331" (id 4) (at 114.935 59.69 0)
       (effects (font (size 1.27 1.27)) hide)
     )
@@
     )
     (path "/a1d92a90-5a32-40f7-9f5c-6fa9bddc0e3b"
-      (reference "C3") (unit 1) (value "470nF/16V") (footprint "Capacitor_SMD:C_0402_1005Metric")
+      (reference "C3") (unit 1) (value "220nF/16V") (footprint "Capacitor_SMD:C_0402_1005Metric")
     )
     (path "/a3aa00f2-727f-4535-9e8a-1d539d2a07f6"
-      (reference "C4") (unit 1) (value "22nF/63V") (footprint "Capacitor_SMD:C_0402_1005Metric")
+      (reference "C4") (unit 1) (value "22nF/50V") (footprint "Capacitor_SMD:C_0402_1005Metric")
     )
     (path "/fc44e920-911b-402f-9258-1d7a939089cc"
@@
     )
     (path "/89235a77-4df8-466c-b78d-c63c56dd3d06"
-      (reference "R5") (unit 1) (value "2.2R") (footprint "Resistor_SMD:R_0402_1005Metric")
+      (reference "R5") (unit 1) (value "1R") (footprint "Resistor_SMD:R_0402_1005Metric")
     )
     (path "/35aa260c-35d5-4a9e-a5ce-23afedc1224d"
